Commit message: with3D

File: nema_description/urdf/arm.xacro (robot description, xacro)
@@ -1,15 +1,15 @@
 <?xml version="1.0"?>
 <robot xmlns:xacro="http://www.ros.org/wiki/xacro">
-    <link name="right_arm1">
+    <link name="right_arm">
         <visual>
-            <origin xyz="0.0 0.0 -0.075" rpy="0.0 0.0 0.0"/>
+            <origin xyz="-0.12 -0.02 -0.35" rpy="0.0 0.0 0.0"/>
             <geometry>
-                <box size="0.050 0.050 0.150"/>
+                <mesh filename="package://nema_description/3D/Mesh/RightArm.dae" scale="0.002 0.002 0.002"/>
             </geometry>
         </visual>
         <collision>
-            <origin xyz="0.0 0.0 -0.075" rpy="0.0 0.0 0.0"/>
+            <origin xyz="-0.12 -0.02 -0.35" rpy="0.0 0.0 0.0"/>
             <geometry>
-                <box size="0.050 0.050 0.150"/>
+                <mesh filename="package://nema_description/3D/Collition/RightArm.stl" scale="0.002 0.002 0.002"/>
             </geometry>
         </collision>
@@ -20,15 +20,29 @@
         </inertial>
     </link>
-    <link name="right_arm2">
+    <link name="right_arm_intermediate_link">
+        <origin xyz="0.0 0.0 0.0" rpy="0.0 0.0 3.14"/>
+        <inertial>
+            <mass value="0.01"/>
+            <inertia ixx="0.0001" ixy="0" ixz="0" iyy="0.0001" iyz="0" izz="0.0001"/>
+        </inertial>
+    </link>
+    <link name="left_arm_intermediate_link">
+        <origin xyz="0.0 0.0 0.0" rpy="0.0 0.0 3.14"/>
+        <inertial>
+            <mass value="0.01"/>
+            <inertia ixx="0.0001" ixy="0" ixz="0" iyy="0.0001" iyz="0" izz="0.0001"/>
+        </inertial>
+    </link>
+    <link name="left_arm">
         <visual>
-            <origin xyz="0.0 0.0 -0.0375" rpy="0.0 0.0 0.0"/>
+            <origin xyz="0.24 0 -0.38" rpy="0.0 0.0 0.0"/>
             <geometry>
-                <box size="0.050 0.050 0.075"/>
+                <mesh filename="package://nema_description/3D/Mesh/LeftArm.dae" scale="0.002 0.002 0.002"/>
             </geometry>
         </visual>
         <collision>
-            <origin xyz="0.0 0.0 -0.0375" rpy="0.0 0.0 0.0"/>
+            <origin xyz="0.24 0 -0.38" rpy="0.0 0.0 0.0"/>
             <geometry>
-                <box size="0.050 0.050 0.075"/>
+                <mesh filename="package://nema_description/3D/Collition/LeftArm.stl" scale="0.002 0.002 0.002"/>
             </geometry>
         </collision>
@@ -39,79 +53,17 @@
         </inertial>
     </link>
-    <link name="right_arm3">
-        <visual>
-            <origin xyz="0.0 0.00 -0.03" rpy="0.0 0.0 0.0"/>
-            <geometry>
-                <box size="0.050 0.050 0.060"/>
-            </geometry>
-        </visual>
-        <collision>
-            <origin xyz="0.0 0.0 -0.03" rpy="0.0 0.0 0.0"/>
-            <geometry>
-                <box size="0.050 0.050 0.060"/>
-            </geometry>
-        </collision>
-        <inertial>
-            <origin xyz="0.0 0.0 -0.030" rpy="0.0 0.0 0.0"/>
-            <mass value="0.01"/>
-            <inertia ixx="0.01" ixy="0.0" ixz="0.0" iyy="0.01" iyz="0.0" izz="0.01"/>
-        </inertial>
-    </link>
-    <link name="left_arm1">
-        <visual>
-            <origin xyz="0.0 0.0 -0.075" rpy="0.0 0.0 0.0"/>
-            <geometry>
-                <box size="0.050 0.050 0.150"/>
-            </geometry>
-        </visual>
-        <collision>
-            <origin xyz="0.0 0.0 -0.075" rpy="0.0 0.0 0.0"/>
-            <geometry>
-                <box size="0.050 0.050 0.150"/>
-            </geometry>
-        </collision>
-        <inertial>
-            <origin xyz="0.0 0.0 -0.075" rpy="0.0 0.0 0.0"/>
-            <mass value="0.06"/>
-            <inertia ixx="0.06" ixy="0.0" ixz="0.0" iyy="0.06" iyz="0.0" izz="0.06"/>
-        </inertial>
-    </link>
-    <link name="left_arm2">
-        <visual>
-            <origin xyz="0.0 0.0 -0.0375" rpy="0.0 0.0 0.0"/>
-            <geometry>
-                <box size="0.050 0.050 0.075"/>
-            </geometry>
-        </visual>
-        <collision>
-            <origin xyz="0.0 0.0 -0.0375" rpy="0.0 0.0 0.0"/>
-            <geometry>
-                <box size="0.050 0.050 0.075"/>
-            </geometry>
-        </collision>
-        <inertial>
-            <origin xyz="0.0 0.0 -0.0375" rpy="0.0 0.0 0.0"/>
-            <mass value="0.03"/>
-            <inertia ixx="0.03" ixy="0.0" ixz="0.0" iyy="0.03" iyz="0.0" izz="0.03"/>
-        </inertial>
-    </link>
-    <link name="left_arm3">
-        <visual>
-            <origin xyz="0.0 0.00 -0.03" rpy="0.0 0.0 0.0"/>
-            <geometry>
-                <box size="0.050 0.050 0.060"/>
-            </geometry>
-        </visual>
-        <collision>
-            <origin xyz="0.0 0.0 -0.03" rpy="0.0 0.0 0.0"/>
-            <geometry>
-                <box size="0.050 0.050 0.060"/>
-            </geometry>
-        </collision>
-        <inertial>
-            <origin xyz="0.0 0.0 -0.030" rpy="0.0 0.0 0.0"/>
-            <mass value="0.01"/>
-            <inertia ixx="0.01" ixy="0.0" ixz="0.0" iyy="0.01" iyz="0.0" izz="0.01"/>
-        </inertial>
-    </link>
+    <xacro:macro name="material_visual" params="ref_link">
+        <gazebo reference="${ref_link}">
+            <visual>
+                <material>
+                    <ambient>0.3 0.3 0.3 1.0</ambient>
+                    <diffuse>0.7 0.7 0.7 1.0</diffuse>
+                    <specular>0.01 0.01 0.01 1.0</specular>
+                    <emissive>0.0 0.0 0.0 1.0</emissive>
+                </material>
+            </visual>
+        </gazebo>
+    </xacro:macro>
+    <xacro:material_visual ref_link="right_arm"/>
+    <xacro:material_visual ref_link="left_arm"/>
 </robot>

File: nema_description/urdf/body.xacro (robot description, xacro)
@@ -6,5 +6,5 @@
             <origin xyz="0.0 0.0 0.050" rpy="0.0 0.0 0.0"/>
             <geometry>
-                <box size="0.350 0.350 0.100"/>
+                <cylinder radius="0.200" length="0.1"/>
             </geometry>
         </visual>
@@ -12,5 +12,5 @@
             <origin xyz="0.0 0.0 0.050" rpy="0.0 0.0 0.0"/>
             <geometry>
-                <box size="0.350 0.350 0.100"/>
+                <cylinder radius="0.200" length="0.1"/>
             </geometry>
         </collision>
@@ -23,17 +23,17 @@
     <link name="body_link">
         <visual>
-            <origin xyz="0.0 0.0 0.200" rpy="0.0 0.0 0.0"/>
+            <origin xyz="0.0 -0.05 -0.010" rpy="0.0 0.0 0.0"/>
             <geometry>
-                <box size="0.350 0.350 0.400"/>
+                <mesh filename="package://nema_description/3D/Mesh/Body.dae" scale="0.002 0.002 0.002"/>
             </geometry>
         </visual>
         <collision>
-            <origin xyz="0.0 0.0 0.200" rpy="0.0 0.0 0.0"/>
+            <origin xyz="0.0 -0.05 -0.010" rpy="0.0 0.0 0.0"/>
             <geometry>
-                <box size="0.350 0.350 0.400"/>
+                <mesh filename="package://nema_description/3D/Collition/Body.stl" scale="0.002 0.002 0.002"/>
             </geometry>
         </collision>
         <inertial>
-            <origin xyz="0 0 0.200" rpy="0.0 0.0 0.0"/>
+            <origin xyz="0 0 0.0" rpy="0.0 0.0 0.0"/>
             <mass value="0.4"/>
             <inertia ixx="0.4" ixy="0.0" ixz="0.0" iyy="0.4" iyz="0.0" izz="0.4"/>
@@ -42,13 +42,13 @@
     <link name="face_link">
         <visual>
-            <origin xyz="0.0 0.0 0.075" rpy="0.0 0.0 0.0"/>
+            <origin xyz="0.0 0.050 -0.470" rpy="0.0 0.0 3.14"/>
             <geometry>
-                <box size="0.200 0.200 0.150"/>
+                <mesh filename="package://nema_description/3D/Mesh/Face.dae" scale="0.002 0.002 0.002"/>
             </geometry>
         </visual>
         <collision>
-            <origin xyz="0.0 0.0 0.075" rpy="0.0 0.0 0.0"/>
+            <origin xyz="0.0 0.050 -0.470" rpy="0.0 0.0 3.14"/>
             <geometry>
-                <box size="0.200 0.200 0.150"/>
+                <mesh filename="package://nema_description/3D/Collition/Face.stl" scale="0.002 0.002 0.002"/>
             </geometry>
         </collision>
@@ -61,8 +61,22 @@
     <link name="face_intermediate_link">
         <inertial>
-            <origin xyz="0 0 0" rpy="0 0 0"/>
-            <mass value="0.0001"/>
-            <inertia ixx="0.0001" ixy="0.0" ixz="0.0" iyy="0.0001" iyz="0.0" izz="0.0001"/>
+            <mass value="0.01"/>
+            <inertia ixx="0.0001" ixy="0" ixz="0" iyy="0.0001" iyz="0" izz="0.0001"/>
         </inertial>
     </link>
+    <xacro:macro name="material_visual" params="ref_link">
+        <gazebo reference="${ref_link}">
+            <visual>
+                <material>
+                    <ambient>0.3 0.3 0.3 1.0</ambient>
+                    <diffuse>0.7 0.7 0.7 1.0</diffuse>
+                    <specular>0.01 0.01 0.01 1.0</specular>
+                    <emissive>0.0 0.0 0.0 1.0</emissive>
+                </material>
+            </visual>
+        </gazebo>
+    </xacro:macro>
+    <xacro:material_visual ref_link="base_link"/>
+    <xacro:material_visual ref_link="body_link"/>
+    <xacro:material_visual ref_link="face_link"/>
 </robot>

File: nema_description/urdf/camera.xacro (robot description, xacro)
@@ -1,3 +1,3 @@
-<?xml version="1.0"?>
+<!-- <?xml version="1.0"?>
 <robot xmlns:xacro="http://www.ros.org/wiki/xacro">
     <joint name="camera_mount_joint" type="fixed">
@@ -61,3 +61,3 @@
         </sensor>
     </gazebo>
-</robot>
+</robot> -->

File: nema_description/urdf/full_xacro_code.xacro (robot description, xacro)
@@ -6,5 +6,5 @@
             <origin xyz="0.0 0.0 0.050" rpy="0.0 0.0 0.0"/>
             <geometry>
-                <box size="0.350 0.350 0.100"/>
+                <cylinder radius="0.200" length="0.1"/>
             </geometry>
         </visual>
@@ -12,6 +12,9 @@
             <origin xyz="0.0 0.0 0.050" rpy="0.0 0.0 0.0"/>
             <geometry>
-                <box size="0.350 0.350 0.100"/>
+                <cylinder radius="0.200" length="0.1"/>
             </geometry>
+            <material name="red">
+                <color rgba="0 0 1 1"/>
+            </material>
         </collision>
         <inertial>
@@ -23,17 +26,17 @@
     <link name="body_link">
         <visual>
-            <origin xyz="0.0 0.0 0.200" rpy="0.0 0.0 0.0"/>
+            <origin xyz="0.0 -0.05 -0.010" rpy="0.0 0.0 0.0"/>
             <geometry>
-                <box size="0.350 0.350 0.400"/>
+                <mesh filename="package://nema_description/3D/Mesh/Body.dae" scale="0.002 0.002 0.002"/>
             </geometry>
         </visual>
         <collision>
-            <origin xyz="0.0 0.0 0.200" rpy="0.0 0.0 0.0"/>
+            <origin xyz="0.0 -0.05 -0.010" rpy="0.0 0.0 0.0"/>
             <geometry>
-                <box size="0.350 0.350 0.400"/>
+                <mesh filename="package://nema_description/3D/Collition/Body.stl" scale="0.002 0.002 0.002"/>
             </geometry>
         </collision>
         <inertial>
-            <origin xyz="0 0 0.200" rpy="0.0 0.0 0.0"/>
+            <origin xyz="0 0 0.0" rpy="0.0 0.0 0.0"/>
             <mass value="0.4"/>
             <inertia ixx="0.4" ixy="0.0" ixz="0.0" iyy="0.4" iyz="0.0" izz="0.4"/>
@@ -42,13 +45,13 @@
     <link name="face_link">
         <visual>
-            <origin xyz="0.0 0.0 0.075" rpy="0.0 0.0 0.0"/>
+            <origin xyz="0.0 0.050 -0.470" rpy="0.0 0.0 3.14"/>
             <geometry>
-                <box size="0.200 0.200 0.150"/>
+                <mesh filename="package://nema_description/3D/Mesh/Face.dae" scale="0.002 0.002 0.002"/>
             </geometry>
         </visual>
         <collision>
-            <origin xyz="0.0 0.0 0.075" rpy="0.0 0.0 0.0"/>
+            <origin xyz="0.0 0.050 -0.470" rpy="0.0 0.0 3.14"/>
             <geometry>
-                <box size="0.200 0.200 0.150"/>
+                <mesh filename="package://nema_description/3D/Collition/Face.stl" scale="0.002 0.002 0.002"/>
             </geometry>
         </collision>
@@ -59,22 +62,16 @@
         </inertial>
     </link>
-    <link name="face_intermediate_link">
-        <inertial>
-            <origin xyz="0 0 0" rpy="0 0 0"/>
-            <mass value="0.0001"/>
-            <inertia ixx="0.0001" ixy="0.0" ixz="0.0" iyy="0.0001" iyz="0.0" izz="0.0001"/>
-        </inertial>
-    </link>
-    <link name="right_arm1">
+    <link name="face_intermediate_link"></link>
+    <link name="right_arm">
         <visual>
-            <origin xyz="0.0 0.0 -0.075" rpy="0.0 0.0 0.0"/>
+            <origin xyz="-0.12 -0.02 -0.35" rpy="0.0 0.0 0.0"/>
             <geometry>
-                <box size="0.050 0.050 0.150"/>
+                <mesh filename="package://nema_description/3D/Mesh/RightArm.dae" scale="0.002 0.002 0.002"/>
             </geometry>
         </visual>
         <collision>
-            <origin xyz="0.0 0.0 -0.075" rpy="0.0 0.0 0.0"/>
+            <origin xyz="-0.12 -0.02 -0.35" rpy="0.0 0.0 0.0"/>
             <geometry>
-                <box size="0.050 0.050 0.150"/>
+                <mesh filename="package://nema_description/3D/Collition/RightArm.stl" scale="0.002 0.002 0.002"/>
             </geometry>
         </collision>
@@ -85,15 +82,21 @@
         </inertial>
     </link>
-    <link name="right_arm2">
+    <link name="right_arm_intermediate_link">
+        <origin xyz="0.0 0.0 0.0" rpy="0.0 0.0 3.14"/>
+    </link>
+    <link name="left_arm_intermediate_link">
+        <origin xyz="0.0 0.0 0.0" rpy="0.0 0.0 3.14"/>
+    </link>
+    <link name="left_arm">
         <visual>
-            <origin xyz="0.0 0.0 -0.0375" rpy="0.0 0.0 0.0"/>
+            <origin xyz="0.24 0 -0.38" rpy="0.0 0.0 0.0"/>
             <geometry>
-                <box size="0.050 0.050 0.075"/>
+                <mesh filename="package://nema_description/3D/Mesh/LeftArm.dae" scale="0.002 0.002 0.002"/>
             </geometry>
         </visual>
         <collision>
-            <origin xyz="0.0 0.0 -0.0375" rpy="0.0 0.0 0.0"/>
+            <origin xyz="0.24 0 -0.38" rpy="0.0 0.0 0.0"/>
             <geometry>
-                <box size="0.050 0.050 0.075"/>
+                <mesh filename="package://nema_description/3D/Collition/LeftArm.stl" scale="0.002 0.002 0.002"/>
             </geometry>
         </collision>
@@ -102,80 +105,4 @@
             <mass value="0.03"/>
             <inertia ixx="0.03" ixy="0.0" ixz="0.0" iyy="0.03" iyz="0.0" izz="0.03"/>
-        </inertial>
-    </link>
-    <link name="right_arm3">
-        <visual>
-            <origin xyz="0.0 0.00 -0.03" rpy="0.0 0.0 0.0"/>
-            <geometry>
-                <box size="0.050 0.050 0.060"/>
-            </geometry>
-        </visual>
-        <collision>
-            <origin xyz="0.0 0.0 -0.03" rpy="0.0 0.0 0.0"/>
-            <geometry>
-                <box size="0.050 0.050 0.060"/>
-            </geometry>
-        </collision>
-        <inertial>
-            <origin xyz="0.0 0.0 -0.030" rpy="0.0 0.0 0.0"/>
-            <mass value="0.01"/>
-            <inertia ixx="0.01" ixy="0.0" ixz="0.0" iyy="0.01" iyz="0.0" izz="0.01"/>
-        </inertial>
-    </link>
-    <link name="left_arm1">
-        <visual>
-            <origin xyz="0.0 0.0 -0.075" rpy="0.0 0.0 0.0"/>
-            <geometry>
-                <box size="0.050 0.050 0.150"/>
-            </geometry>
-        </visual>
-        <collision>
-            <origin xyz="0.0 0.0 -0.075" rpy="0.0 0.0 0.0"/>
-            <geometry>
-                <box size="0.050 0.050 0.150"/>
-            </geometry>
-        </collision>
-        <inertial>
-            <origin xyz="0.0 0.0 -0.075" rpy="0.0 0.0 0.0"/>
-            <mass value="0.06"/>
-            <inertia ixx="0.06" ixy="0.0" ixz="0.0" iyy="0.06" iyz="0.0" izz="0.06"/>
-        </inertial>
-    </link>
-    <link name="left_arm2">
-        <visual>
-            <origin xyz="0.0 0.0 -0.0375" rpy="0.0 0.0 0.0"/>
-            <geometry>
-                <box size="0.050 0.050 0.075"/>
-            </geometry>
-        </visual>
-        <collision>
-            <origin xyz="0.0 0.0 -0.0375" rpy="0.0 0.0 0.0"/>
-            <geometry>
-                <box size="0.050 0.050 0.075"/>
-            </geometry>
-        </collision>
-        <inertial>
-            <origin xyz="0.0 0.0 -0.0375" rpy="0.0 0.0 0.0"/>
-            <mass value="0.03"/>
-            <inertia ixx="0.03" ixy="0.0" ixz="0.0" iyy="0.03" iyz="0.0" izz="0.03"/>
-        </inertial>
-    </link>
-    <link name="left_arm3">
-        <visual>
-            <origin xyz="0.0 0.00 -0.03" rpy="0.0 0.0 0.0"/>
-            <geometry>
-                <box size="0.050 0.050 0.060"/>
-            </geometry>
-        </visual>
-        <collision>
-            <origin xyz="0.0 0.0 -0.03" rpy="0.0 0.0 0.0"/>
-            <geometry>
-                <box size="0.050 0.050 0.060"/>
-            </geometry>
-        </collision>
-        <inertial>
-            <origin xyz="0.0 0.0 -0.030" rpy="0.0 0.0 0.0"/>
-            <mass value="0.01"/>
-            <inertia ixx="0.01" ixy="0.0" ixz="0.0" iyy="0.01" iyz="0.0" izz="0.01"/>
         </inertial>
     </link>
@@ -191,5 +118,5 @@
         <child link="body_link"/>
         <axis xyz="0 0 1"/>
-        <limit effort="30.0" lower="-0.85" upper="0.85" velocity="10.0"/>
+        <limit effort="5" lower="-0.85" upper="0.85" velocity="0.3"/>
     </joint>
     <joint name="face_joint_z" type="revolute">
@@ -207,86 +134,37 @@
         <child link="face_link"/>
         <axis xyz="1 0 0"/>
-        <limit effort="30.0" lower="-0.85" upper="0.85" velocity="10.0"/>
+        <limit effort="5" lower="-0.85" upper="0.85" velocity="0.25"/>
     </joint>
-    <joint name="right_joint1" type="revolute">
+    <joint name="right_joint_y" type="revolute">
+        <safety_controller k_position="100.0" k_velocity="40.0" soft_lower_limit="0" soft_upper_limit="0.4"/>
+        <origin rpy="0.0 0 0" xyz="0.125 -0.03 0.300"/>
+        <parent link="body_link"/>
+        <child link="right_arm_intermediate_link"/>
+        <axis xyz="0 1 0"/>
+        <limit effort="30.0" lower="-0.05" upper="0.45" velocity="10.0"/>
+    </joint>
+    <joint name="right_joint_x" type="revolute">
         <safety_controller k_position="100.0" k_velocity="40.0" soft_lower_limit="0" soft_upper_limit="0.8"/>
-        <origin rpy="0.02 0 0" xyz="0.200 0 0.300"/>
-        <parent link="body_link"/>
-        <child link="right_arm1"/>
+        <origin rpy="0.0 0 0" xyz="0.0 0 0.0"/>
+        <parent link="right_arm_intermediate_link"/>
+        <child link="right_arm"/>
         <axis xyz="1 0 0"/>
         <limit effort="30.0" lower="-0.05" upper="0.85" velocity="10.0"/>
     </joint>
-    <joint name="right_joint2" type="revolute">
+    <joint name="left_joint_y" type="revolute">
+        <safety_controller k_position="100.0" k_velocity="40.0" soft_lower_limit="0" soft_upper_limit="0.8"/>
+        <origin rpy="0.0 0 0" xyz="-0.125 -0.03 0.300"/>
+        <parent link="body_link"/>
+        <child link="left_arm_intermediate_link"/>
+        <axis xyz="0 1 0"/>
+        <limit effort="30.0" lower="-0.05" upper="0.85" velocity="10.0"/>
+    </joint>
+    <joint name="left_joint_x" type="revolute">
         <safety_controller k_position="100.0" k_velocity="40.0" soft_lower_limit="0" soft_upper_limit="0.4"/>
-        <origin rpy="0.02 0 0" xyz="0.050 0 -0.125"/>
-        <parent link="right_arm1"/>
-        <child link="right_arm2"/>
+        <origin rpy="0.0 0 0" xyz="0.0 0 0.0"/>
+        <parent link="left_arm_intermediate_link"/>
+        <child link="left_arm"/>
         <axis xyz="1 0 0"/>
         <limit effort="30.0" lower="-0.05" upper="0.45" velocity="10.0"/>
     </joint>
-    <joint name="right_joint3" type="revolute">
-        <safety_controller k_position="100.0" k_velocity="40.0" soft_lower_limit="0" soft_upper_limit="0.2"/>
-        <origin rpy="0.02 0 0" xyz="0.050 0 -0.055"/>
-        <parent link="right_arm2"/>
-        <child link="right_arm3"/>
-        <axis xyz="1 0 0"/>
-        <limit effort="30.0" lower="-0.05" upper="0.25" velocity="10.0"/>
-    </joint>
-    <joint name="left_joint1" type="revolute">
-        <safety_controller k_position="100.0" k_velocity="40.0" soft_lower_limit="0" soft_upper_limit="0.8"/>
-        <origin rpy="0.02 0 0" xyz="-0.200 0 0.300"/>
-        <parent link="body_link"/>
-        <child link="left_arm1"/>
-        <axis xyz="1 0 0"/>
-        <limit effort="30.0" lower="-0.05" upper="0.85" velocity="10.0"/>
-    </joint>
-    <joint name="left_joint2" type="revolute">
-        <safety_controller k_position="100.0" k_velocity="40.0" soft_lower_limit="0" soft_upper_limit="0.4"/>
-        <origin rpy="0.02 0 0" xyz="-0.050 0 -0.125"/>
-        <parent link="left_arm1"/>
-        <child link="left_arm2"/>
-        <axis xyz="1 0 0"/>
-        <limit effort="30.0" lower="-0.05" upper="0.45" velocity="10.0"/>
-    </joint>
-    <joint name="left_joint3" type="revolute">
-        <safety_controller k_position="100.0" k_velocity="40.0" soft_lower_limit="0" soft_upper_limit="0.2"/>
-        <origin rpy="0.02 0 0" xyz="-0.050 0 -0.055"/>
-        <parent link="left_arm2"/>
-        <child link="left_arm3"/>
-        <axis xyz="1 0 0"/>
-        <limit effort="30.0" lower="-0.05" upper="0.25" velocity="10.0"/>
-    </joint>
-    <joint name="camera_mount_joint" type="fixed">
-        <parent link="body_link"/>
-        <child link="camera_link"/>
-        <origin xyz="0.0 0.195 0.100" rpy="0 0 0"/>
-    </joint>
-    <link name="camera_link">
-        <inertial>
-            <mass value="0.1"/>
-            <origin xyz="0 0 0"/>
-            <inertia ixx="0.001" iyy="0.001" izz="0.001"
-                    ixy="0" ixz="0" iyz="0"/>
-        </inertial>
-        <visual>
-            <origin xyz="0 0 0" rpy="0 0 0"/>
-            <geometry>
-                <box size="0.04 0.04 0.04"/>
-            </geometry>
-            <material name="green">
-                <color rgba= "0 1 0 1"/>
-            </material>
-        </visual>
-        <collision>
-            <geometry>
-                <box size="0.04 0.04 0.04"/>
-            </geometry>
-        </collision>
-    </link>
-    <link name="camera_optical_link"/>
-    <joint name="camera_optical_joint" type="fixed">
-        <parent link="camera_link"/>
-        <child link="camera_optical_link"/>
-        <origin xyz="0 0 0" rpy="-1.5708 0 -1.5708"/>
-    </joint>
 </robot>
