Commit message: with3D

File: nema_description/urdf/joints.xacro (robot description, xacro)
@@ -30,51 +30,35 @@
         <limit effort="5" lower="-0.85" upper="0.85" velocity="0.25"/>
     </joint>
-    <joint name="right_joint1" type="revolute">
+    <joint name="right_joint_y" type="revolute">
+        <safety_controller k_position="100.0" k_velocity="40.0" soft_lower_limit="0" soft_upper_limit="0.4"/>
+        <origin rpy="0.0 0 0" xyz="0.125 -0.03 0.300"/>
+        <parent link="body_link"/>
+        <child link="right_arm_intermediate_link"/>
+        <axis xyz="0 1 0"/>
+        <limit effort="30.0" lower="-0.05" upper="0.45" velocity="10.0"/>
+    </joint>
+    <joint name="right_joint_x" type="revolute">
         <safety_controller k_position="100.0" k_velocity="40.0" soft_lower_limit="0" soft_upper_limit="0.8"/>
-        <origin rpy="0.02 0 0" xyz="0.200 0 0.300"/>
-        <parent link="body_link"/>
-        <child link="right_arm1"/>
+        <origin rpy="0.0 0 0" xyz="0.0 0 0.0"/>
+        <parent link="right_arm_intermediate_link"/>
+        <child link="right_arm"/>
         <axis xyz="1 0 0"/>
         <limit effort="30.0" lower="-0.05" upper="0.85" velocity="10.0"/>
     </joint>
-    <joint name="right_joint2" type="revolute">
+    <joint name="left_joint_y" type="revolute">
+        <safety_controller k_position="100.0" k_velocity="40.0" soft_lower_limit="0" soft_upper_limit="0.8"/>
+        <origin rpy="0.0 0 0" xyz="-0.125 -0.03 0.300"/>
+        <parent link="body_link"/>
+        <child link="left_arm_intermediate_link"/>
+        <axis xyz="0 1 0"/>
+        <limit effort="30.0" lower="-0.05" upper="0.85" velocity="10.0"/>
+    </joint>
+    <joint name="left_joint_x" type="revolute">
         <safety_controller k_position="100.0" k_velocity="40.0" soft_lower_limit="0" soft_upper_limit="0.4"/>
-        <origin rpy="0.02 0 0" xyz="0.050 0 -0.125"/>
-        <parent link="right_arm1"/>
-        <child link="right_arm2"/>
+        <origin rpy="0.0 0 0" xyz="0.0 0 0.0"/>
+        <parent link="left_arm_intermediate_link"/>
+        <child link="left_arm"/>
         <axis xyz="1 0 0"/>
         <limit effort="30.0" lower="-0.05" upper="0.45" velocity="10.0"/>
     </joint>
-    <joint name="right_joint3" type="revolute">
-        <safety_controller k_position="100.0" k_velocity="40.0" soft_lower_limit="0" soft_upper_limit="0.2"/>
-        <origin rpy="0.02 0 0" xyz="0.050 0 -0.055"/>
-        <parent link="right_arm2"/>
-        <child link="right_arm3"/>
-        <axis xyz="1 0 0"/>
-        <limit effort="30.0" lower="-0.05" upper="0.25" velocity="10.0"/>
-    </joint>
-    <joint name="left_joint1" type="revolute">
-        <safety_controller k_position="100.0" k_velocity="40.0" soft_lower_limit="0" soft_upper_limit="0.8"/>
-        <origin rpy="0.02 0 0" xyz="-0.200 0 0.300"/>
-        <parent link="body_link"/>
-        <child link="left_arm1"/>
-        <axis xyz="1 0 0"/>
-        <limit effort="30.0" lower="-0.05" upper="0.85" velocity="10.0"/>
-    </joint>
-    <joint name="left_joint2" type="revolute">
-        <safety_controller k_position="100.0" k_velocity="40.0" soft_lower_limit="0" soft_upper_limit="0.4"/>
-        <origin rpy="0.02 0 0" xyz="-0.050 0 -0.125"/>
-        <parent link="left_arm1"/>
-        <child link="left_arm2"/>
-        <axis xyz="1 0 0"/>
-        <limit effort="30.0" lower="-0.05" upper="0.45" velocity="10.0"/>
-    </joint>
-    <joint name="left_joint3" type="revolute">
-        <safety_controller k_position="100.0" k_velocity="40.0" soft_lower_limit="0" soft_upper_limit="0.2"/>
-        <origin rpy="0.02 0 0" xyz="-0.050 0 -0.055"/>
-        <parent link="left_arm2"/>
-        <child link="left_arm3"/>
-        <axis xyz="1 0 0"/>
-        <limit effort="30.0" lower="-0.05" upper="0.25" velocity="10.0"/>
-    </joint>
 </robot>

File: nema_description/urdf/model.urdf.xacro (robot description, xacro)
@@ -4,5 +4,5 @@
     <xacro:include filename="$(find nema_description)/urdf/arm.xacro" />
     <xacro:include filename="$(find nema_description)/urdf/joints.xacro" />
-    <xacro:include filename="$(find nema_description)/urdf/camera.xacro" />
+    <!-- <xacro:include filename="$(find nema_description)/urdf/camera.xacro" /> -->
     <xacro:include filename="$(find nema_description)/urdf/gazebo.xacro" />
     <xacro:include filename="$(find nema_description)/urdf/robot_controllers.xacro" />

File: nema_description/urdf/robot_controllers.xacro (robot description, xacro)
@@ -12,6 +12,4 @@
                 <param name="max">0.85</param>
             </command_interface>
-            <command_interface name="velocity"/>
-            <command_interface name="acceleration"/>
             <state_interface name="position">
                 <param name="initial_value">0</param>
@@ -23,6 +21,34 @@
                 <param name="max">0.85</param>
             </command_interface>
-            <command_interface name="velocity"/>
-            <command_interface name="acceleration"/>
+            <state_interface name="position">
+                <param name="initial_value">0</param>
+            </state_interface>
+        </joint>
+        <!-- Joint 3 -->
+        <joint name="left_joint_x">
+            <command_interface name="position">
+                <param name="min">-0.05</param>
+                <param name="max">0.45</param>
+            </command_interface>
+            <state_interface name="position">
+                <param name="initial_value">0</param>
+            </state_interface>
+        </joint>
+        <!-- Joint 5 -->
+        <joint name="left_joint_y">
+            <command_interface name="position">
+                <param name="min">-0.05</param>
+                <param name="max">0.85</param>
+            </command_interface>
+            <state_interface name="position">
+                <param name="initial_value">0</param>
+            </state_interface>
+        </joint>
+        <!-- Joint 3 -->
+        <joint name="right_joint_x">
+            <command_interface name="position">
+                <param name="min">-0.05</param>
+                <param name="max">0.45</param>
+            </command_interface>
             <state_interface name="position">
                 <param name="initial_value">0</param>
@@ -30,71 +56,9 @@
         </joint>
         <!-- Joint 2 -->
-        <joint name="right_joint1">
+        <joint name="right_joint_y">
             <command_interface name="position">
                 <param name="min">-0.05</param>
                 <param name="max">0.85</param>
             </command_interface>
-            <command_interface name="velocity"/>
-            <command_interface name="acceleration"/>
-            <state_interface name="position">
-                <param name="initial_value">0</param>
-            </state_interface>
-        </joint>
-        <!-- Joint 3 -->
-        <joint name="right_joint2">
-            <command_interface name="position">
-                <param name="min">-0.05</param>
-                <param name="max">0.45</param>
-            </command_interface>
-            <command_interface name="velocity"/>
-            <command_interface name="acceleration"/>
-            <state_interface name="position">
-                <param name="initial_value">0</param>
-            </state_interface>
-        </joint>
-        <!-- Joint 4 -->
-        <joint name="right_joint3">
-            <command_interface name="position">
-                <param name="min">-0.05</param>
-                <param name="max">0.25</param>
-            </command_interface>
-            <command_interface name="velocity"/>
-            <command_interface name="acceleration"/>
-            <state_interface name="position">
-                <param name="initial_value">0</param>
-            </state_interface>
-        </joint>
-        <!-- Joint 5 -->
-        <joint name="left_joint1">
-            <command_interface name="position">
-                <param name="min">-0.05</param>
-                <param name="max">0.85</param>
-            </command_interface>
-            <command_interface name="velocity"/>
-            <command_interface name="acceleration"/>
-            <state_interface name="position">
-                <param name="initial_value">0</param>
-            </state_interface>
-        </joint>
-        <!-- Joint 3 -->
-        <joint name="left_joint2">
-            <command_interface name="position">
-                <param name="min">-0.05</param>
-                <param name="max">0.45</param>
-            </command_interface>
-            <command_interface name="velocity"/>
-            <command_interface name="acceleration"/>
-            <state_interface name="position">
-                <param name="initial_value">0</param>
-            </state_interface>
-        </joint>
-        <!-- Joint 4 -->
-        <joint name="left_joint3">
-            <command_interface name="position">
-                <param name="min">-0.05</param>
-                <param name="max">0.25</param>
-            </command_interface>
-            <command_interface name="velocity"/>
-            <command_interface name="acceleration"/>
             <state_interface name="position">
                 <param name="initial_value">0</param>
@@ -102,3 +66,23 @@
         </joint>
     </ros2_control>
+    <!-- <transmission name="body_joint_trans">
+            <plugin>transmission_interface/SimpleTransmission</plugin>
+            <joint name="body_joint">
+                <hardwareInterface>hardware_interface/PositionJointInterface</hardwareInterface>
+            </joint>
+            <actuator name="body_motor">
+                <hardwareInterface>hardware_interface/PositionJointInterface</hardwareInterface>
+                <mechanicalReduction>1</mechanicalReduction>
+            </actuator>
+        </transmission>
+        <transmission name="face_joint_x_trans">
+            <plugin>transmission_interface/SimpleTransmission</plugin>
+            <joint name="face_joint_x">
+                <hardwareInterface>hardware_interface/PositionJointInterface</hardwareInterface>
+            </joint>
+            <actuator name="face_motor">
+                <hardwareInterface>hardware_interface/PositionJointInterface</hardwareInterface>
+                <mechanicalReduction>1</mechanicalReduction>
+            </actuator>
+        </transmission> -->
 </robot>
