Commit message: nema_gazebo

File: nema_description/urdf/robot_controllers.xacro (robot description, xacro)
@@ -17,4 +17,13 @@
         </joint>
         <joint name="face_joint_x">
+            <command_interface name="position">
+                <param name="min">-0.85</param>
+                <param name="max">0.85</param>
+            </command_interface>
+            <state_interface name="position">
+                <param name="initial_value">0</param>
+            </state_interface>
+        </joint>
+        <joint name="face_joint_z">
             <command_interface name="position">
                 <param name="min">-0.85</param>
