Commit message: PI_works

File: nema_description/urdf/body.xacro (robot description, xacro)
@@ -8,4 +8,7 @@
                 <cylinder radius="0.200" length="0.1"/>
             </geometry>
+	    <material name="red">
+       		<color rgba="1 0 0 1"/>
+    	    </material>
         </visual>
         <collision>

File: nema_description/urdf/gazebo.xacro (robot description, xacro)
@@ -4,4 +4,6 @@
         <plugin filename="gz_ros2_control-system" name="gz_ros2_control::GazeboSimROS2ControlPlugin">
             <parameters>$(find nema_gazebo)/config/ros2_controllers.yaml</parameters>
+	    <robot_param>robot_description</robot_param>
+            <robot_param_node>robot_state_publisher</robot_param_node>
         </plugin>
         <plugin filename="gz-sim-sensors-system" name="gz::sim::systems::Sensors">

File: nema_description/urdf/model.urdf.xacro (robot description, xacro)
@@ -4,5 +4,5 @@
     <xacro:include filename="$(find nema_description)/urdf/arm.xacro" />
     <xacro:include filename="$(find nema_description)/urdf/joints.xacro" />
-    <!-- <xacro:include filename="$(find nema_description)/urdf/camera.xacro" /> -->
+    <!--<xacro:include filename="$(find nema_description)/urdf/camera.xacro" />-->
     <xacro:include filename="$(find nema_description)/urdf/gazebo.xacro" />
     <xacro:include filename="$(find nema_description)/urdf/robot_controllers.xacro" />
